Commit message: started moveit2 integration

File: alpha_description/gazebo/alpha.gazebo.xacro (robot description, xacro)
@@ -6,5 +6,5 @@
       <plugin name="gazebo_ros2_control" filename="libgazebo_ros2_control.so">
         <parameters>
-          $(find alpha_bringup)/config/alpha_controllers.yaml</parameters>
+          $(find alpha_description)/config/alpha_controllers.yaml</parameters>
       </plugin>
     </gazebo>

File: alpha_description/urdf/alpha.urdf.xacro (robot description, xacro)
@@ -1,37 +1,160 @@
 <?xml version="1.0"?>
-<robot name="alpha" xmlns:xacro="http://ros.org/wiki/xacro">
-  <!-- Declare arguments which can be set from a launch file -->
-  <xacro:arg name="prefix" default="" />
-  <xacro:arg name="use_gazebo" default="true" />
-  <xacro:arg name="use_fake_hardware" default="true" />
-  <xacro:arg name="mock_sensor_commands" default="true" />
-  <xacro:arg name="serial_port" default="" />
-  <xacro:arg name="heartbeat_timeout" default="5000" />
-  <xacro:arg name="state_update_frequency" default="200" />
-  <!-- Import Alpha macro -->
-  <xacro:include
-    filename="$(find alpha_description)/urdf/alpha_description.urdf.xacro" />
-  <!-- Import ros2_control macro -->
-  <xacro:include
-    filename="$(find alpha_description)/ros2_control/alpha.ros2_control.xacro" />
-  <xacro:if value="$(arg use_gazebo)">
+<robot xmlns:xacro="http://ros.org/wiki/xacro">
+  <xacro:macro name="alpha" params="parent prefix *origin">
+    <joint name="${prefix}base_joint" type="fixed">
+      <xacro:insert_block name="origin" />
+      <parent link="${parent}" />
+      <child link="${prefix}base_link" />
+      <origin xyz="0 0 0" rpy="0 0 0" />
+    </joint>
+    <material name="${prefix}black">
+      <color rgba="0.3 0.3 0.3 1" />
+    </material>
+    <link name="${prefix}base_link" />
+    <link name="${prefix}m3_inline_link">
+      <visual>
+        <geometry>
+          <mesh filename="package://alpha_description/meshes/M3-INLINE.stl" />
+        </geometry>
+        <origin rpy="0 0 0" xyz="0 0 0" />
+        <material name="${prefix}black" />
+      </visual>
+      <collision>
+        <geometry>
+          <cylinder length="0.150" radius="0.020" />
+        </geometry>
+        <origin rpy="0 1.57075 0" xyz="-0.075 0 0" />
+      </collision>
+    </link>
+    <joint name="${prefix}base_link_joint" type="fixed">
+      <parent link="${prefix}base_link" />
+      <child link="${prefix}m3_inline_link" />
+      <origin rpy="0 0 0" />
+    </joint>
+    <link name="${prefix}m2_1_1_link">
+      <visual>
+        <geometry>
+          <mesh filename="package://alpha_description/meshes/M2-1-1.stl" />
+        </geometry>
+        <origin rpy="0 0 0" xyz="0 0 0" />
+        <material name="${prefix}black" />
+      </visual>
+      <collision>
+        <geometry>
+          <cylinder length="0.066" radius="0.020" />
+        </geometry>
+        <origin rpy="0 0 0" xyz="0 0 0.000" />
+      </collision>
+    </link>
+    <joint name="${prefix}axis_e" type="revolute">
+      <parent link="${prefix}m3_inline_link" />
+      <child link="${prefix}m2_1_1_link" />
+      <origin xyz="0 0 0.014" />
+      <axis xyz="0 0 1" />
+      <limit effort="9.0" lower="0.0" upper="6.3" velocity="0.5" />
+    </joint>
+    <link name="${prefix}m2_joint_link">
+      <visual>
+        <geometry>
+          <mesh filename="package://alpha_description/meshes/M2.stl" />
+        </geometry>
+        <origin rpy="0 0 0" xyz="0 0 0" />
+        <material name="${prefix}black" />
+      </visual>
+      <collision>
+        <geometry>
+          <cylinder length="0.145" radius="0.020" />
+        </geometry>
+        <origin rpy="0 0 0" xyz="-0.02 0 -0.0725" />
+      </collision>
+      <collision>
+        <geometry>
+          <cylinder length="0.040" radius="0.020" />
+        </geometry>
+        <origin rpy="1.5707 0 0" xyz="0 0 0" />
+      </collision>
+      <collision>
+        <geometry>
+          <cylinder length="0.040" radius="0.020" />
+        </geometry>
+        <origin rpy="1.5707 0 0" xyz="-0.040 0 -0.1453" />
+      </collision>
+    </link>
+    <joint name="${prefix}axis_d" type="revolute">
+      <parent link="${prefix}m2_1_1_link" />
+      <child link="${prefix}m2_joint_link" />
+      <origin xyz="-0.02 0 0.033" />
+      <axis xyz="0 1 0" />
+      <limit effort="9.0" lower="0.0" upper="3.8" velocity="0.5" />
+    </joint>
+    <link name="${prefix}m2_1_2_link">
+      <visual>
+        <geometry>
+          <mesh filename="package://alpha_description/meshes/M2-1-3.stl" />
+        </geometry>
+        <origin rpy="0 0 0" xyz="0 0 0" />
+        <material name="${prefix}black" />
+      </visual>
+      <collision>
+        <geometry>
+          <cylinder length="0.033" radius="0.020" />
+        </geometry>
+        <origin rpy="0 0 0" xyz="0.02 0 0.0165" />
+      </collision>
+    </link>
+    <joint name="${prefix}axis_c" type="revolute">
+      <parent link="${prefix}m2_joint_link" />
+      <child link="${prefix}m2_1_2_link" />
+      <origin xyz="-0.04 0 -0.1453" rpy="0 0 3.14159" />
+      <axis xyz="0 1 0" />
+      <limit effort="9.0" lower="0.0" upper="3.5" velocity="0.5" />
+    </joint>
+    <link name="${prefix}m1_link">
+      <visual>
+        <geometry>
+          <mesh
+            filename="package://alpha_description/meshes/RS1-100-101-123.stl" />
+        </geometry>
+        <origin rpy="0 -1.5707 0" xyz="0 0 0" />
+        <material name="${prefix}black" />
+      </visual>
+      <collision>
+        <geometry>
+          <cylinder length="0.10975" radius="0.020" />
+        </geometry>
+        <origin rpy="0 0 0" xyz="0.00 0 0.054875" />
+      </collision>
+    </link>
+    <joint name="${prefix}axis_b" type="revolute">
+      <parent link="${prefix}m2_1_2_link" />
+      <child link="${prefix}m1_link" />
+      <origin xyz="0.02 0 0.033" rpy="0 0 2.09439" />
+      <axis xyz="0 0 -1" />
+      <limit effort="9.0" lower="0.0" upper="6.2" velocity="0.5" />
+    </joint>
+    <material name="${prefix}ee_black">
+      <color rgba="0.3 0.3 0.3 1" />
+    </material>
+    <joint name="${prefix}ee_joint" type="fixed">
+      <origin rpy="0 0 0" xyz="0 0 0.09975" />
+      <parent link="${prefix}m1_link" />
+      <child link="${prefix}ee_base_link" />
+    </joint>
+    <link name="${prefix}ee_base_link" />
+    <link name="${prefix}push_rod" />
+    <joint name="${prefix}axis_a" type="prismatic">
+      <origin rpy="0 0 0" xyz="0 0 0.009" />
+      <parent link="${prefix}ee_base_link" />
+      <child link="${prefix}push_rod" />
+      <axis xyz="0 0 1" />
+      <limit effort="10" lower="0" upper="0.015" velocity="10" />
+    </joint>
     <xacro:include
-      filename="$(find alpha_description)/gazebo/alpha.gazebo.xacro" />
-  </xacro:if>
-  <link name="world" />
-  <xacro:alpha_robot parent="world" prefix="$(arg prefix)">
-    <origin xyz="0 0 0" rpy="0 0 0" />
-  </xacro:alpha_robot>
-  <xacro:alpha_system prefix="$(arg prefix)"
-    use_fake_hardware="$(arg use_fake_hardware)"
-    mock_sensor_commands="$(arg mock_sensor_commands)"
-    serial_port="$(arg serial_port)"
-    heartbeat_timeout="$(arg heartbeat_timeout)"
-    state_update_frequency="$(arg state_update_frequency)" />
-  <xacro:if value="$(arg use_gazebo)">
-    <gazebo reference="world">
-      <static>true</static>
-    </gazebo>
-    <xacro:alpha_gazebo prefix="$(arg prefix)" />
-  </xacro:if>
+      filename="$(find alpha_description)/urdf/end_effectors/standard_jaws.urdf.xacro" />
+    <xacro:alpha_standard_jaws parent="${prefix}ee_base_link"
+      prefix="${prefix}standard_jaws_"
+      axis_a="${prefix}axis_a">
+      <origin xyz="0 0 0" rpy="0 0 0" />
+    </xacro:alpha_standard_jaws>
+  </xacro:macro>
 </robot>

Commit message: debugging gazebo

File: alpha_description/gazebo/alpha.gazebo.xacro (robot description, xacro)
@@ -15,4 +15,38 @@
       </plugin>
     </gazebo>
+    <gazebo reference="${prefix}base_link">
+      <material>Gazebo/Gray</material>
+    </gazebo>
+    <gazebo reference="${prefix}ee_base_link">
+      <material>Gazebo/Gray</material>
+    </gazebo>
+    <gazebo reference="${prefix}m1_link" />
+    <gazebo reference="${prefix}m1_link">
+      <material>Gazebo/Gray</material>
+    </gazebo>
+    <gazebo reference="${prefix}m2_1_1_link">
+      <material>Gazebo/Gray</material>
+    </gazebo>
+    <gazebo reference="${prefix}m2_1_2_link">
+      <material>Gazebo/Gray</material>
+    </gazebo>
+    <gazebo reference="${prefix}m2_joint_link">
+      <material>Gazebo/Gray</material>
+    </gazebo>
+    <gazebo reference="${prefix}m3_inline_link">
+      <material>Gazebo/Gray</material>
+    </gazebo>
+    <gazebo reference="${prefix}push_rod">
+      <material>Gazebo/Gray</material>
+    </gazebo>
+    <gazebo reference="${prefix}standard_jaws_base_link">
+      <material>Gazebo/Gray</material>
+    </gazebo>
+    <gazebo reference="${prefix}standard_jaws_rs1_130_link">
+      <material>Gazebo/Gray</material>
+    </gazebo>
+    <gazebo reference="${prefix}standard_jaws_rs1_139_link">
+      <material>Gazebo/Gray</material>
+    </gazebo>
   </xacro:macro>
 </robot>

File: alpha_description/ros2_control/alpha.ros2_control.xacro (robot description, xacro)
@@ -13,15 +13,17 @@
         </hardware>
       </xacro:if>
-      <hardware>
-        <xacro:if value="${use_fake_hardware}">
-          <plugin>mock_components/GenericSystem</plugin>
-        </xacro:if>
-        <xacro:unless value="${use_fake_hardware}">
-          <plugin>alpha_hardware/AlphaHardware</plugin>
-          <param name="serial_port">${serial_port}</param>
-          <param name="heartbeat_timeout">${heartbeat_timeout}</param>
-          <param name="state_update_frequency">${state_update_frequency}</param>
-        </xacro:unless>
-      </hardware>
+      <xacro:unless value="$(arg use_sim)">
+        <hardware>
+          <xacro:if value="${use_fake_hardware}">
+            <plugin>mock_components/GenericSystem</plugin>
+          </xacro:if>
+          <xacro:unless value="${use_fake_hardware}">
+            <plugin>alpha_hardware/AlphaHardware</plugin>
+            <param name="serial_port">${serial_port}</param>
+            <param name="heartbeat_timeout">${heartbeat_timeout}</param>
+            <param name="state_update_frequency">${state_update_frequency}</param>
+          </xacro:unless>
+        </hardware>
+      </xacro:unless>
       <joint name="axis_e">
         <command_interface name="position" />

File: alpha_description/urdf/alpha.urdf.xacro (robot description, xacro)
@@ -26,4 +26,9 @@
         <origin rpy="0 1.57075 0" xyz="-0.075 0 0" />
       </collision>
+      <inertial>
+        <mass value="2e-06" />
+        <inertia ixx="1.1e-09" ixy="0" ixz="0" iyy="1.1e-09" iyz="0"
+          izz="1.1e-09" />
+      </inertial>
     </link>
     <joint name="${prefix}base_link_joint" type="fixed">
@@ -46,4 +51,9 @@
         <origin rpy="0 0 0" xyz="0 0 0.000" />
       </collision>
+      <inertial>
+        <mass value="2e-06" />
+        <inertia ixx="1.1e-09" ixy="0" ixz="0" iyy="1.1e-09" iyz="0"
+          izz="1.1e-09" />
+      </inertial>
     </link>
     <joint name="${prefix}axis_e" type="revolute">
@@ -80,4 +90,9 @@
         <origin rpy="1.5707 0 0" xyz="-0.040 0 -0.1453" />
       </collision>
+      <inertial>
+        <mass value="2e-06" />
+        <inertia ixx="1.1e-09" ixy="0" ixz="0" iyy="1.1e-09" iyz="0"
+          izz="1.1e-09" />
+      </inertial>
     </link>
     <joint name="${prefix}axis_d" type="revolute">
@@ -102,4 +117,9 @@
         <origin rpy="0 0 0" xyz="0.02 0 0.0165" />
       </collision>
+      <inertial>
+        <mass value="2e-06" />
+        <inertia ixx="1.1e-09" ixy="0" ixz="0" iyy="1.1e-09" iyz="0"
+          izz="1.1e-09" />
+      </inertial>
     </link>
     <joint name="${prefix}axis_c" type="revolute">
@@ -125,4 +145,9 @@
         <origin rpy="0 0 0" xyz="0.00 0 0.054875" />
       </collision>
+      <inertial>
+        <mass value="2e-06" />
+        <inertia ixx="1.1e-09" ixy="0" ixz="0" iyy="1.1e-09" iyz="0"
+          izz="1.1e-09" />
+      </inertial>
     </link>
     <joint name="${prefix}axis_b" type="revolute">
@@ -141,6 +166,18 @@
       <child link="${prefix}ee_base_link" />
     </joint>
-    <link name="${prefix}ee_base_link" />
-    <link name="${prefix}push_rod" />
+    <link name="${prefix}ee_base_link">
+      <inertial>
+        <mass value="2e-06" />
+        <inertia ixx="1.1e-09" ixy="0" ixz="0" iyy="1.1e-09" iyz="0"
+          izz="1.1e-09" />
+      </inertial>
+    </link>
+    <link name="${prefix}push_rod">
+      <inertial>
+        <mass value="2e-06" />
+        <inertia ixx="1.1e-09" ixy="0" ixz="0" iyy="1.1e-09" iyz="0"
+          izz="1.1e-09" />
+      </inertial>
+    </link>
     <joint name="${prefix}axis_a" type="prismatic">
       <origin rpy="0 0 0" xyz="0 0 0.009" />

File: alpha_description/urdf/end_effectors/standard_jaws.urdf.xacro (robot description, xacro)
@@ -36,4 +36,9 @@
         <origin xyz="0.0 -0.008 0.045" rpy="0 0 0" />
       </collision>
+      <inertial>
+        <mass value="2e-06" />
+        <inertia ixx="1.1e-09" ixy="0" ixz="0" iyy="1.1e-09" iyz="0"
+          izz="1.1e-09" />
+      </inertial>
     </link>
     <joint name="${prefix}rs1_130_joint" type="revolute">
@@ -60,4 +65,9 @@
         <origin xyz="0.0 0.008 0.045" rpy="0 0 0" />
       </collision>
+      <inertial>
+        <mass value="2e-06" />
+        <inertia ixx="1.1e-09" ixy="0" ixz="0" iyy="1.1e-09" iyz="0"
+          izz="1.1e-09" />
+      </inertial>
     </link>
     <joint name="${prefix}rs1_139_joint" type="revolute">
