Commit message: save point for ramen

File: alpha_description/srdf/alpha.srdf.xacro (robot description, xacro)
@@ -8,9 +8,8 @@
             <joint name="${prefix}axis_c" />
             <joint name="${prefix}axis_b" />
-        </group>
-        <group name="${prefix}jaws">
             <joint name="${prefix}axis_a" />
         </group>
         <group_state name="home" group="${prefix}arm">
+            <joint name="${prefix}axis_a" value="0" />
             <joint name="${prefix}axis_b" value="0" />
             <joint name="${prefix}axis_c" value="0" />
@@ -18,6 +17,4 @@
             <joint name="${prefix}axis_e" value="0" />
         </group_state>
-        <end_effector name="${prefix}jaws" parent_link="${prefix}ee_base_link"
-            group="${prefix}jaws" />
         <passive_joint name="${prefix}standard_jaws_rs1_130_joint" />
         <passive_joint name="${prefix}standard_jaws_rs1_139_joint" />
