Commit message: Starting to migrate moveit2 configs to description package

File: alpha_description/config/alpha.config.xacro (robot description, xacro)
@@ -3,4 +3,5 @@
   <!-- Declare arguments which can be set from a launch file -->
   <xacro:arg name="prefix" default="" />
+  <xacro:arg name="use_sim" default="false" />
   <xacro:arg name="use_fake_hardware" default="true" />
   <xacro:arg name="mock_sensor_commands" default="true" />
@@ -14,4 +15,9 @@
   <xacro:include
     filename="$(find alpha_description)/ros2_control/alpha.ros2_control.xacro" />
+  <!-- Import Gazebo macro -->
+  <xacro:if value="$(arg use_sim)">
+    <xacro:include
+      filename="$(find alpha_description)/gazebo/alpha.gazebo.xacro" />
+  </xacro:if>
   <link name="world" />
   <xacro:alpha parent="world" prefix="$(arg prefix)">
@@ -24,3 +30,9 @@
     heartbeat_timeout="$(arg heartbeat_timeout)"
     state_update_frequency="$(arg state_update_frequency)" />
+  <xacro:if value="$(arg use_sim)">
+    <gazebo reference="world">
+      <static>true</static>
+    </gazebo>
+    <xacro:alpha_gazebo prefix="$(arg prefix)" />
+  </xacro:if>
 </robot>

File: alpha_description/ros2_control/alpha.ros2_control.xacro (robot description, xacro)
@@ -1,12 +1,17 @@
 <?xml version="1.0"?>
 <robot xmlns:xacro="http://www.ros.org/wiki/xacro">
-  <xacro:macro name="alpha_system"
-    params="prefix use_fake_hardware mock_sensor_commands serial_port heartbeat_timeout state_update_frequency">
-    <ros2_control name="${prefix}alpha_hardware" type="system">
+  <xacro:macro name="alpha_ros2_control"
+    params="name prefix serial_port heartbeat_timeout state_update_frequency initial_positions_file use_sim:=^|false use_fake_hardware:=^true">
+    <xacro:property name="initial_positions"
+      value="${load_yaml(initial_positions_file)['initial_positions']}" />
+    <ros2_control name="${name}" type="system">
+      <xacro:if value="$(arg use_sim)">
+        <hardware>
+          <plugin>gazebo_ros2_control/GazeboSystem</plugin>
+        </hardware>
+      </xacro:if>
       <hardware>
         <xacro:if value="${use_fake_hardware}">
           <plugin>mock_components/GenericSystem</plugin>
-          <param name="mock_sensor_commands">${mock_sensor_commands}</param>
-          <param name="state_following_offset">0.0</param>
         </xacro:if>
         <xacro:unless value="${use_fake_hardware}">
@@ -17,5 +22,6 @@
         </xacro:unless>
       </hardware>
-      <joint name="${prefix}axis_e">
+      <joint name="axis_e">
+        <param name="initial_value">${initial_positions['axis_e']}</param>
         <command_interface name="position" />
         <command_interface name="velocity" />
@@ -23,5 +29,6 @@
         <state_interface name="velocity" />
       </joint>
-      <joint name="${prefix}axis_d">
+      <joint name="axis_d">
+        <param name="initial_value">${initial_positions['axis_d']}</param>
         <command_interface name="position" />
         <command_interface name="velocity" />
@@ -29,5 +36,6 @@
         <state_interface name="velocity" />
       </joint>
-      <joint name="${prefix}axis_c">
+      <joint name="axis_c">
+        <param name="initial_value">${initial_positions['axis_c']}</param>
         <command_interface name="position" />
         <command_interface name="velocity" />
@@ -35,5 +43,6 @@
         <state_interface name="velocity" />
       </joint>
-      <joint name="${prefix}axis_b">
+      <joint name="axis_b">
+        <param name="initial_value">${initial_positions['axis_b']}</param>
         <command_interface name="position" />
         <command_interface name="velocity" />
@@ -41,5 +50,6 @@
         <state_interface name="velocity" />
       </joint>
-      <joint name="${prefix}axis_a">
+      <joint name="axis_a">
+        <param name="initial_value">${initial_positions['axis_a']}</param>
         <command_interface name="position" />
         <command_interface name="velocity" />

File: alpha_description/urdf/alpha.urdf.xacro (robot description, xacro)
@@ -52,5 +52,5 @@
       <origin xyz="0 0 0.014" />
       <axis xyz="0 0 1" />
-      <limit effort="9.0" lower="0.0" upper="6.3" velocity="0.5" />
+      <limit effort="9.0" lower="0.0" upper="6.10" velocity="0.5" />
     </joint>
     <link name="${prefix}m2_joint_link">
@@ -86,5 +86,5 @@
       <origin xyz="-0.02 0 0.033" />
       <axis xyz="0 1 0" />
-      <limit effort="9.0" lower="0.0" upper="3.8" velocity="0.5" />
+      <limit effort="9.0" lower="0.0" upper="3.49" velocity="0.5" />
     </joint>
     <link name="${prefix}m2_1_2_link">
@@ -108,5 +108,5 @@
       <origin xyz="-0.04 0 -0.1453" rpy="0 0 3.14159" />
       <axis xyz="0 1 0" />
-      <limit effort="9.0" lower="0.0" upper="3.5" velocity="0.5" />
+      <limit effort="9.0" lower="0.0" upper="3.22" velocity="0.5" />
     </joint>
     <link name="${prefix}m1_link">
@@ -131,5 +131,5 @@
       <origin xyz="0.02 0 0.033" rpy="0 0 2.09439" />
       <axis xyz="0 0 -1" />
-      <limit effort="9.0" lower="0.0" upper="6.2" velocity="0.5" />
+      <limit effort="9.0" lower="0.0" upper="3.22" velocity="0.5" />
     </joint>
     <material name="${prefix}ee_black">

File: alpha_moveit2_config/config/alpha.ros2_control.xacro (robot description, xacro)
@@ -1,52 +1,54 @@
 <?xml version="1.0"?>
 <robot xmlns:xacro="http://www.ros.org/wiki/xacro">
-    <xacro:macro name="alpha_ros2_control" params="name initial_positions_file">
-        <xacro:property name="initial_positions" value="${load_yaml(initial_positions_file)['initial_positions']}"/>
-        <ros2_control name="${name}" type="system">
-            <hardware>
-                <!-- By default, set up controllers for simulation. This won't work on real hardware -->
-                <plugin>mock_components/GenericSystem</plugin>
-            </hardware>
-            <joint name="axis_e">
-                <command_interface name="position"/>
-                <command_interface name="velocity"/>
-                <state_interface name="position">
-                  <param name="initial_value">${initial_positions['axis_e']}</param>
-                </state_interface>
-                <state_interface name="velocity"/>
-            </joint>
-            <joint name="axis_d">
-                <command_interface name="position"/>
-                <command_interface name="velocity"/>
-                <state_interface name="position">
-                  <param name="initial_value">${initial_positions['axis_d']}</param>
-                </state_interface>
-                <state_interface name="velocity"/>
-            </joint>
-            <joint name="axis_c">
-                <command_interface name="position"/>
-                <command_interface name="velocity"/>
-                <state_interface name="position">
-                  <param name="initial_value">${initial_positions['axis_c']}</param>
-                </state_interface>
-                <state_interface name="velocity"/>
-            </joint>
-            <joint name="axis_b">
-                <command_interface name="position"/>
-                <command_interface name="velocity"/>
-                <state_interface name="position">
-                  <param name="initial_value">${initial_positions['axis_b']}</param>
-                </state_interface>
-                <state_interface name="velocity"/>
-            </joint>
-            <joint name="axis_a">
-                <command_interface name="position"/>
-                <command_interface name="velocity"/>
-                <state_interface name="position">
-                  <param name="initial_value">${initial_positions['axis_a']}</param>
-                </state_interface>
-                <state_interface name="velocity"/>
-            </joint>
-        </ros2_control>
-    </xacro:macro>
+  <xacro:macro name="alpha_ros2_control" params="name initial_positions_file">
+    <xacro:property name="initial_positions"
+      value="${load_yaml(initial_positions_file)['initial_positions']}" />
+    <ros2_control name="${name}" type="system">
+      <hardware>
+        <!-- By default, set up controllers for simulation. This won't work on
+        real hardware -->
+        <plugin>mock_components/GenericSystem</plugin>
+      </hardware>
+      <joint name="axis_e">
+        <command_interface name="position" />
+        <command_interface name="velocity" />
+        <state_interface name="position">
+          <param name="initial_value">${initial_positions['axis_e']}</param>
+        </state_interface>
+        <state_interface name="velocity" />
+      </joint>
+      <joint name="axis_d">
+        <command_interface name="position" />
+        <command_interface name="velocity" />
+        <state_interface name="position">
+          <param name="initial_value">${initial_positions['axis_d']}</param>
+        </state_interface>
+        <state_interface name="velocity" />
+      </joint>
+      <joint name="axis_c">
+        <command_interface name="position" />
+        <command_interface name="velocity" />
+        <state_interface name="position">
+          <param name="initial_value">${initial_positions['axis_c']}</param>
+        </state_interface>
+        <state_interface name="velocity" />
+      </joint>
+      <joint name="axis_b">
+        <command_interface name="position" />
+        <command_interface name="velocity" />
+        <state_interface name="position">
+          <param name="initial_value">${initial_positions['axis_b']}</param>
+        </state_interface>
+        <state_interface name="velocity" />
+      </joint>
+      <joint name="axis_a">
+        <command_interface name="position" />
+        <command_interface name="velocity" />
+        <state_interface name="position">
+          <param name="initial_value">${initial_positions['axis_a']}</param>
+        </state_interface>
+        <state_interface name="velocity" />
+      </joint>
+    </ros2_control>
+  </xacro:macro>
 </robot>

Commit message: started working on adding launch files

File: alpha_description/config/alpha.config.xacro (robot description, xacro)
@@ -5,8 +5,9 @@
   <xacro:arg name="use_sim" default="false" />
   <xacro:arg name="use_fake_hardware" default="true" />
-  <xacro:arg name="mock_sensor_commands" default="true" />
   <xacro:arg name="serial_port" default="" />
   <xacro:arg name="heartbeat_timeout" default="5000" />
   <xacro:arg name="state_update_frequency" default="200" />
+  <xacro:arg name="controllers_file" default="alpha_controllers.yaml" />
+  <xacro:arg name="initial_positions_file" default="initial_positions.yaml" />
   <!-- Import Alpha macro -->
   <xacro:include
@@ -16,23 +17,20 @@
     filename="$(find alpha_description)/ros2_control/alpha.ros2_control.xacro" />
   <!-- Import Gazebo macro -->
-  <xacro:if value="$(arg use_sim)">
-    <xacro:include
-      filename="$(find alpha_description)/gazebo/alpha.gazebo.xacro" />
-  </xacro:if>
+  <xacro:include
+    filename="$(find alpha_description)/gazebo/alpha.gazebo.xacro" />
   <link name="world" />
   <xacro:alpha parent="world" prefix="$(arg prefix)">
     <origin xyz="0 0 0" rpy="0 0 0" />
   </xacro:alpha>
-  <xacro:alpha_system prefix="$(arg prefix)"
-    use_fake_hardware="$(arg use_fake_hardware)"
-    mock_sensor_commands="$(arg mock_sensor_commands)"
+  <xacro:alpha_system prefix="$(arg prefix)" name="ReachAlpha5"
+    use_fake_hardware="$(arg use_fake_hardware)" use_sim="$(arg use_sim)"
     serial_port="$(arg serial_port)"
     heartbeat_timeout="$(arg heartbeat_timeout)"
-    state_update_frequency="$(arg state_update_frequency)" />
-  <xacro:if value="$(arg use_sim)">
-    <gazebo reference="world">
-      <static>true</static>
-    </gazebo>
-    <xacro:alpha_gazebo prefix="$(arg prefix)" />
-  </xacro:if>
+    state_update_frequency="$(arg state_update_frequency)"
+    initial_positions_file="$(arg initial_positions_file)" />
+  <gazebo reference="world">
+    <static>true</static>
+  </gazebo>
+  <xacro:alpha_gazebo prefix="$(arg prefix)"
+    controllers_file="$(arg controllers_file)" />
 </robot>

File: alpha_description/gazebo/alpha.gazebo.xacro (robot description, xacro)
@@ -1,10 +1,10 @@
 <?xml version="1.0"?>
 <robot xmlns:xacro="http://ros.org/wiki/xacro">
-  <xacro:macro name="alpha_gazebo" params="prefix">
+  <xacro:macro name="alpha_gazebo" params="prefix controllers_file">
     <!-- ros_control plugin -->
     <gazebo>
       <plugin name="gazebo_ros2_control" filename="libgazebo_ros2_control.so">
         <parameters>
-          $(find alpha_description)/config/alpha_controllers.yaml</parameters>
+          $(find alpha_description)/config/${controllers_file}</parameters>
       </plugin>
     </gazebo>

File: alpha_description/ros2_control/alpha.ros2_control.xacro (robot description, xacro)
@@ -1,5 +1,5 @@
 <?xml version="1.0"?>
 <robot xmlns:xacro="http://www.ros.org/wiki/xacro">
-  <xacro:macro name="alpha_ros2_control"
+  <xacro:macro name="alpha_system"
     params="name prefix serial_port heartbeat_timeout state_update_frequency initial_positions_file use_sim:=^|false use_fake_hardware:=^true">
     <xacro:property name="initial_positions"

Commit message: Fixed moveit configs

File: alpha_description/config/alpha.config.xacro (robot description, xacro)
@@ -20,7 +20,7 @@
     filename="$(find alpha_description)/gazebo/alpha.gazebo.xacro" />
   <link name="world" />
-  <xacro:alpha parent="world" prefix="$(arg prefix)">
+  <xacro:alpha_urdf parent="world" prefix="$(arg prefix)">
     <origin xyz="0 0 0" rpy="0 0 0" />
-  </xacro:alpha>
+  </xacro:alpha_urdf>
   <xacro:alpha_system prefix="$(arg prefix)" name="ReachAlpha5"
     use_fake_hardware="$(arg use_fake_hardware)" use_sim="$(arg use_sim)"

File: alpha_description/urdf/alpha.urdf.xacro (robot description, xacro)
@@ -1,5 +1,5 @@
 <?xml version="1.0"?>
 <robot xmlns:xacro="http://ros.org/wiki/xacro">
-  <xacro:macro name="alpha" params="parent prefix *origin">
+  <xacro:macro name="alpha_urdf" params="parent prefix *origin">
     <joint name="${prefix}base_joint" type="fixed">
       <xacro:insert_block name="origin" />

Commit message: fixed controller execution

File: alpha_description/config/alpha.config.xacro (robot description, xacro)
@@ -2,5 +2,4 @@
 <robot name="alpha" xmlns:xacro="http://ros.org/wiki/xacro">
   <!-- Declare arguments which can be set from a launch file -->
-  <xacro:arg name="prefix" default="" />
   <xacro:arg name="use_sim" default="false" />
   <xacro:arg name="use_fake_hardware" default="true" />
@@ -10,4 +9,7 @@
   <xacro:arg name="controllers_file" default="alpha_controllers.yaml" />
   <xacro:arg name="initial_positions_file" default="initial_positions.yaml" />
+  <xacro:arg name="initial_velocities_file" default="initial_velocities.yaml" />
+  <xacro:arg name="namespace" default="/" />
+  <xacro:arg name="prefix" default="" />
   <!-- Import Alpha macro -->
   <xacro:include
@@ -23,4 +25,7 @@
     <origin xyz="0 0 0" rpy="0 0 0" />
   </xacro:alpha_urdf>
+  <gazebo reference="world">
+    <static>true</static>
+  </gazebo>
   <xacro:alpha_system prefix="$(arg prefix)" name="ReachAlpha5"
     use_fake_hardware="$(arg use_fake_hardware)" use_sim="$(arg use_sim)"
@@ -28,9 +33,7 @@
     heartbeat_timeout="$(arg heartbeat_timeout)"
     state_update_frequency="$(arg state_update_frequency)"
-    initial_positions_file="$(arg initial_positions_file)" />
-  <gazebo reference="world">
-    <static>true</static>
-  </gazebo>
+    initial_positions_file="$(arg initial_positions_file)"
+    initial_velocities_file="$(arg initial_velocities_file)" />
   <xacro:alpha_gazebo prefix="$(arg prefix)"
-    controllers_file="$(arg controllers_file)" />
+    controllers_file="$(arg controllers_file)" namespace="$(arg namespace)" />
 </robot>

File: alpha_description/gazebo/alpha.gazebo.xacro (robot description, xacro)
@@ -1,24 +1,18 @@
 <?xml version="1.0"?>
 <robot xmlns:xacro="http://ros.org/wiki/xacro">
-  <xacro:macro name="alpha_gazebo" params="prefix controllers_file">
+  <xacro:macro name="alpha_gazebo" params="prefix controllers_file namespace">
     <!-- ros_control plugin -->
     <gazebo>
       <plugin name="gazebo_ros2_control" filename="libgazebo_ros2_control.so">
-        <robot_param_node>robot_state_publisher</robot_param_node>
+        <xacro:if value="${namespace != '/'}">
+          <ros>
+            <namespace>/${namespace[:-1]}</namespace>
+          </ros>
+          <robot_param_node>/${namespace}robot_state_publisher</robot_param_node>
+        </xacro:if>
         <parameters>
           $(find alpha_description)/config/${controllers_file}</parameters>
       </plugin>
     </gazebo>
-    <gazebo reference="${prefix}base_link" />
-    <gazebo reference="${prefix}ee_base_link" />
-    <gazebo reference="${prefix}m1_link" />
-    <gazebo reference="${prefix}m2_1_1_link" />
-    <gazebo reference="${prefix}m2_1_2_link" />
-    <gazebo reference="${prefix}m2_joint_link" />
-    <gazebo reference="${prefix}m3_inline_link" />
-    <gazebo reference="${prefix}push_rod" />
-    <gazebo reference="${prefix}standard_jaws_base_link" />
-    <gazebo reference="${prefix}standard_jaws_rs1_130_link" />
-    <gazebo reference="${prefix}standard_jaws_rs1_139_link" />
   </xacro:macro>
 </robot>

File: alpha_description/ros2_control/alpha.ros2_control.xacro (robot description, xacro)
@@ -2,7 +2,9 @@
 <robot xmlns:xacro="http://www.ros.org/wiki/xacro">
   <xacro:macro name="alpha_system"
-    params="name prefix serial_port heartbeat_timeout state_update_frequency initial_positions_file use_sim:=^|false use_fake_hardware:=^true">
+    params="name prefix serial_port heartbeat_timeout state_update_frequency initial_positions_file initial_velocities_file use_sim:=^|false  use_fake_hardware:=^true">
     <xacro:property name="initial_positions"
       value="${xacro.load_yaml(initial_positions_file)['initial_positions']}" />
+    <xacro:property name="initial_velocities"
+      value="${xacro.load_yaml(initial_velocities_file)['initial_velocities']}" />
     <ros2_control name="${name}" type="system">
       <xacro:if value="$(arg use_sim)">
@@ -25,45 +27,50 @@
         <command_interface name="position" />
         <command_interface name="velocity" />
-        <state_interface name="position" />
         <state_interface name="position">
           <param name="initial_value">${initial_positions['axis_e']}</param>
         </state_interface>
-        <state_interface name="velocity" />
+        <state_interface name="velocity">
+          <param name="initial_value">${initial_velocities['axis_e']}</param>
+        </state_interface>
       </joint>
       <joint name="axis_d">
         <command_interface name="position" />
         <command_interface name="velocity" />
-        <state_interface name="position" />
         <state_interface name="position">
           <param name="initial_value">${initial_positions['axis_d']}</param>
         </state_interface>
-        <state_interface name="velocity" />
+        <state_interface name="velocity">
+          <param name="initial_value">${initial_velocities['axis_d']}</param>
+        </state_interface>
       </joint>
       <joint name="axis_c">
         <command_interface name="position" />
         <command_interface name="velocity" />
-        <state_interface name="position" />
         <state_interface name="position">
           <param name="initial_value">${initial_positions['axis_c']}</param>
         </state_interface>
-        <state_interface name="velocity" />
+        <state_interface name="velocity">
+          <param name="initial_value">${initial_velocities['axis_c']}</param>
+        </state_interface>
       </joint>
       <joint name="axis_b">
         <command_interface name="position" />
         <command_interface name="velocity" />
-        <state_interface name="position" />
         <state_interface name="position">
           <param name="initial_value">${initial_positions['axis_b']}</param>
         </state_interface>
-        <state_interface name="velocity" />
+        <state_interface name="velocity">
+          <param name="initial_value">${initial_velocities['axis_b']}</param>
+        </state_interface>
       </joint>
       <joint name="axis_a">
         <command_interface name="position" />
         <command_interface name="velocity" />
-        <state_interface name="position" />
         <state_interface name="position">
           <param name="initial_value">${initial_positions['axis_a']}</param>
         </state_interface>
-        <state_interface name="velocity" />
+        <state_interface name="velocity">
+          <param name="initial_value">${initial_velocities['axis_a']}</param>
+        </state_interface>
       </joint>
     </ros2_control>
