Commit message: Removed gazebo stuff for time being

File: alpha_description/config/alpha.config.xacro (robot description, xacro)
@@ -2,5 +2,4 @@
 <robot name="alpha" xmlns:xacro="http://ros.org/wiki/xacro">
   <!-- Declare arguments which can be set from a launch file -->
-  <xacro:arg name="use_sim" default="false" />
   <xacro:arg name="use_fake_hardware" default="true" />
   <xacro:arg name="serial_port" default="" />
@@ -29,5 +28,5 @@
   </gazebo>
   <xacro:alpha_system prefix="$(arg prefix)" name="ReachAlpha5"
-    use_fake_hardware="$(arg use_fake_hardware)" use_sim="$(arg use_sim)"
+    use_fake_hardware="$(arg use_fake_hardware)"
     serial_port="$(arg serial_port)"
     heartbeat_timeout="$(arg heartbeat_timeout)"

File: alpha_description/ros2_control/alpha.ros2_control.xacro (robot description, xacro)
@@ -8,22 +8,15 @@
       value="${xacro.load_yaml(initial_velocities_file)['initial_velocities']}" />
     <ros2_control name="${name}" type="system">
-      <xacro:if value="$(arg use_sim)">
-        <hardware>
-          <plugin>gazebo_ros2_control/GazeboSystem</plugin>
-        </hardware>
-      </xacro:if>
-      <xacro:unless value="$(arg use_sim)">
-        <hardware>
-          <xacro:if value="${use_fake_hardware}">
-            <plugin>mock_components/GenericSystem</plugin>
-          </xacro:if>
-          <xacro:unless value="${use_fake_hardware}">
-            <plugin>alpha_hardware/AlphaHardware</plugin>
-            <param name="serial_port">${serial_port}</param>
-            <param name="heartbeat_timeout">${heartbeat_timeout}</param>
-            <param name="state_update_frequency">${state_update_frequency}</param>
-          </xacro:unless>
-        </hardware>
-      </xacro:unless>
+      <hardware>
+        <xacro:if value="${use_fake_hardware}">
+          <plugin>mock_components/GenericSystem</plugin>
+        </xacro:if>
+        <xacro:unless value="${use_fake_hardware}">
+          <plugin>alpha_hardware/AlphaHardware</plugin>
+          <param name="serial_port">${serial_port}</param>
+          <param name="heartbeat_timeout">${heartbeat_timeout}</param>
+          <param name="state_update_frequency">${state_update_frequency}</param>
+        </xacro:unless>
+      </hardware>
       <joint name="axis_e">
         <command_interface name="position" />

File: alpha_description/urdf/alpha.urdf.xacro (robot description, xacro)
@@ -26,9 +26,4 @@
         <origin rpy="0 1.57075 0" xyz="-0.075 0 0" />
       </collision>
-      <inertial>
-        <mass value="2e-06" />
-        <inertia ixx="1.1e-09" ixy="0" ixz="0" iyy="1.1e-09" iyz="0"
-          izz="1.1e-09" />
-      </inertial>
     </link>
     <joint name="${prefix}base_link_joint" type="fixed">
@@ -51,9 +46,4 @@
         <origin rpy="0 0 0" xyz="0 0 0.000" />
       </collision>
-      <inertial>
-        <mass value="2e-06" />
-        <inertia ixx="1.1e-09" ixy="0" ixz="0" iyy="1.1e-09" iyz="0"
-          izz="1.1e-09" />
-      </inertial>
     </link>
     <joint name="${prefix}axis_e" type="revolute">
@@ -90,9 +80,4 @@
         <origin rpy="1.5707 0 0" xyz="-0.040 0 -0.1453" />
       </collision>
-      <inertial>
-        <mass value="2e-06" />
-        <inertia ixx="1.1e-09" ixy="0" ixz="0" iyy="1.1e-09" iyz="0"
-          izz="1.1e-09" />
-      </inertial>
     </link>
     <joint name="${prefix}axis_d" type="revolute">
@@ -117,9 +102,4 @@
         <origin rpy="0 0 0" xyz="0.02 0 0.0165" />
       </collision>
-      <inertial>
-        <mass value="2e-06" />
-        <inertia ixx="1.1e-09" ixy="0" ixz="0" iyy="1.1e-09" iyz="0"
-          izz="1.1e-09" />
-      </inertial>
     </link>
     <joint name="${prefix}axis_c" type="revolute">
@@ -145,9 +125,4 @@
         <origin rpy="0 0 0" xyz="0.00 0 0.054875" />
       </collision>
-      <inertial>
-        <mass value="2e-06" />
-        <inertia ixx="1.1e-09" ixy="0" ixz="0" iyy="1.1e-09" iyz="0"
-          izz="1.1e-09" />
-      </inertial>
     </link>
     <joint name="${prefix}axis_b" type="revolute">
@@ -166,18 +141,6 @@
       <child link="${prefix}ee_base_link" />
     </joint>
-    <link name="${prefix}ee_base_link">
-      <inertial>
-        <mass value="2e-06" />
-        <inertia ixx="1.1e-09" ixy="0" ixz="0" iyy="1.1e-09" iyz="0"
-          izz="1.1e-09" />
-      </inertial>
-    </link>
-    <link name="${prefix}push_rod">
-      <inertial>
-        <mass value="2e-06" />
-        <inertia ixx="1.1e-09" ixy="0" ixz="0" iyy="1.1e-09" iyz="0"
-          izz="1.1e-09" />
-      </inertial>
-    </link>
+    <link name="${prefix}ee_base_link" />
+    <link name="${prefix}push_rod" />
     <joint name="${prefix}axis_a" type="prismatic">
       <origin rpy="0 0 0" xyz="0 0 0.009" />

File: alpha_description/urdf/end_effectors/standard_jaws.urdf.xacro (robot description, xacro)
@@ -36,9 +36,4 @@
         <origin xyz="0.0 -0.008 0.045" rpy="0 0 0" />
       </collision>
-      <inertial>
-        <mass value="2e-06" />
-        <inertia ixx="1.1e-09" ixy="0" ixz="0" iyy="1.1e-09" iyz="0"
-          izz="1.1e-09" />
-      </inertial>
     </link>
     <joint name="${prefix}rs1_130_joint" type="revolute">
@@ -65,9 +60,4 @@
         <origin xyz="0.0 0.008 0.045" rpy="0 0 0" />
       </collision>
-      <inertial>
-        <mass value="2e-06" />
-        <inertia ixx="1.1e-09" ixy="0" ixz="0" iyy="1.1e-09" iyz="0"
-          izz="1.1e-09" />
-      </inertial>
     </link>
     <joint name="${prefix}rs1_139_joint" type="revolute">

Commit message: IMPORTANT GAZEBO SAVE POINT

File: alpha_description/config/alpha.config.xacro (robot description, xacro)
@@ -3,4 +3,5 @@
   <!-- Declare arguments which can be set from a launch file -->
   <xacro:arg name="use_fake_hardware" default="true" />
+  <xacro:arg name="use_sim" default="false" />
   <xacro:arg name="serial_port" default="" />
   <xacro:arg name="heartbeat_timeout" default="5000" />
@@ -17,4 +18,7 @@
   <xacro:include
     filename="$(find alpha_description)/ros2_control/alpha.ros2_control.xacro" />
+  <!-- Import Gazebo macro -->
+  <xacro:include
+    filename="$(find alpha_description)/gazebo/alpha.gazebo.xacro" />
   <link name="world" />
   <xacro:alpha_urdf parent="world" prefix="$(arg prefix)">
@@ -30,4 +34,7 @@
     state_update_frequency="$(arg state_update_frequency)"
     initial_positions_file="$(arg initial_positions_file)"
-    initial_velocities_file="$(arg initial_velocities_file)" />
+    initial_velocities_file="$(arg initial_velocities_file)"
+    use_sim="$(arg use_sim)" />
+  <xacro:alpha_gazebo prefix="$(arg prefix)"
+    controllers_file="$(arg controllers_file)" namespace="$(arg namespace)" />
 </robot>

File: alpha_description/ros2_control/alpha.ros2_control.xacro (robot description, xacro)
@@ -2,5 +2,5 @@
 <robot xmlns:xacro="http://www.ros.org/wiki/xacro">
   <xacro:macro name="alpha_system"
-    params="name prefix serial_port heartbeat_timeout state_update_frequency initial_positions_file initial_velocities_file use_fake_hardware:=^true">
+    params="name prefix serial_port heartbeat_timeout state_update_frequency initial_positions_file initial_velocities_file use_sim:=^|false  use_fake_hardware:=^true">
     <xacro:property name="initial_positions"
       value="${xacro.load_yaml(initial_positions_file)['initial_positions']}" />
@@ -8,15 +8,22 @@
       value="${xacro.load_yaml(initial_velocities_file)['initial_velocities']}" />
     <ros2_control name="${name}" type="system">
-      <hardware>
-        <xacro:if value="${use_fake_hardware}">
-          <plugin>mock_components/GenericSystem</plugin>
-        </xacro:if>
-        <xacro:unless value="${use_fake_hardware}">
-          <plugin>alpha_hardware/AlphaHardware</plugin>
-          <param name="serial_port">${serial_port}</param>
-          <param name="heartbeat_timeout">${heartbeat_timeout}</param>
-          <param name="state_update_frequency">${state_update_frequency}</param>
-        </xacro:unless>
-      </hardware>
+      <xacro:if value="$(arg use_sim)">
+        <hardware>
+          <plugin>gazebo_ros2_control/GazeboSystem</plugin>
+        </hardware>
+      </xacro:if>
+      <xacro:unless value="$(arg use_sim)">
+        <hardware>
+          <xacro:if value="${use_fake_hardware}">
+            <plugin>mock_components/GenericSystem</plugin>
+          </xacro:if>
+          <xacro:unless value="${use_fake_hardware}">
+            <plugin>alpha_hardware/AlphaHardware</plugin>
+            <param name="serial_port">${serial_port}</param>
+            <param name="heartbeat_timeout">${heartbeat_timeout}</param>
+            <param name="state_update_frequency">${state_update_frequency}</param>
+          </xacro:unless>
+        </hardware>
+      </xacro:unless>
       <joint name="axis_e">
         <command_interface name="position" />

File: alpha_description/urdf/end_effectors/standard_jaws.urdf.xacro (robot description, xacro)
@@ -20,4 +20,9 @@
         <material name="${prefix}black" />
       </visual>
+      <inertial>
+        <mass value="2e-06" />
+        <inertia ixx="1.1e-09" ixy="0" ixz="0" iyy="1.1e-09" iyz="0"
+          izz="1.1e-09" />
+      </inertial>
     </link>
     <link name="${prefix}rs1_130_link">
@@ -36,4 +41,9 @@
         <origin xyz="0.0 -0.008 0.045" rpy="0 0 0" />
       </collision>
+      <inertial>
+        <mass value="2e-06" />
+        <inertia ixx="1.1e-09" ixy="0" ixz="0" iyy="1.1e-09" iyz="0"
+          izz="1.1e-09" />
+      </inertial>
     </link>
     <joint name="${prefix}rs1_130_joint" type="revolute">
@@ -60,4 +70,9 @@
         <origin xyz="0.0 0.008 0.045" rpy="0 0 0" />
       </collision>
+      <inertial>
+        <mass value="2e-06" />
+        <inertia ixx="1.1e-09" ixy="0" ixz="0" iyy="1.1e-09" iyz="0"
+          izz="1.1e-09" />
+      </inertial>
     </link>
     <joint name="${prefix}rs1_139_joint" type="revolute">

Commit message: Resolved *most* of the comments from the pr review

File: alpha_description/config/alpha.config.xacro (robot description, xacro)
@@ -5,6 +5,5 @@
   <xacro:arg name="use_sim" default="false" />
   <xacro:arg name="serial_port" default="" />
-  <xacro:arg name="heartbeat_timeout" default="5000" />
-  <xacro:arg name="state_update_frequency" default="200" />
+  <xacro:arg name="state_update_frequency" default="250" />
   <xacro:arg name="controllers_file" default="alpha_controllers.yaml" />
   <xacro:arg name="initial_positions_file" default="initial_positions.yaml" />
@@ -31,5 +30,4 @@
     use_fake_hardware="$(arg use_fake_hardware)"
     serial_port="$(arg serial_port)"
-    heartbeat_timeout="$(arg heartbeat_timeout)"
     state_update_frequency="$(arg state_update_frequency)"
     initial_positions_file="$(arg initial_positions_file)"

File: alpha_description/ros2_control/alpha.ros2_control.xacro (robot description, xacro)
@@ -2,5 +2,5 @@
 <robot xmlns:xacro="http://www.ros.org/wiki/xacro">
   <xacro:macro name="alpha_system"
-    params="name prefix serial_port heartbeat_timeout state_update_frequency initial_positions_file initial_velocities_file use_sim:=^|false  use_fake_hardware:=^true">
+    params="name prefix serial_port state_update_frequency initial_positions_file initial_velocities_file use_sim:=^|false  use_fake_hardware:=^true">
     <xacro:property name="initial_positions"
       value="${xacro.load_yaml(initial_positions_file)['initial_positions']}" />
@@ -21,5 +21,4 @@
             <plugin>alpha_hardware/AlphaHardware</plugin>
             <param name="serial_port">${serial_port}</param>
-            <param name="heartbeat_timeout">${heartbeat_timeout}</param>
             <param name="state_update_frequency">${state_update_frequency}</param>
           </xacro:unless>

File: alpha_description/srdf/alpha.srdf.xacro (robot description, xacro)
@@ -2,5 +2,5 @@
 <robot xmlns:xacro="http://www.ros.org/wiki/xacro">
     <xacro:macro name="alpha_srdf" params="prefix">
-        <group name="${prefix}arm">
+        <group name="${prefix}alpha">
             <link name="${prefix}ee_base_link" />
             <joint name="${prefix}axis_e" />
@@ -10,9 +10,9 @@
             <joint name="${prefix}axis_a" />
         </group>
-        <group_state name="home" group="${prefix}arm">
+        <group_state name="home" group="${prefix}alpha">
             <joint name="${prefix}axis_a" value="0" />
-            <joint name="${prefix}axis_b" value="0" />
+            <joint name="${prefix}axis_b" value="1.5746" />
             <joint name="${prefix}axis_c" value="0" />
-            <joint name="${prefix}axis_d" value="1.5746" />
+            <joint name="${prefix}axis_d" value="0" />
             <joint name="${prefix}axis_e" value="0" />
         </group_state>
