Commit message: fixed joint limit issues

File: alpha_description/ros2_control/alpha.ros2_control.xacro (robot description, xacro)
@@ -13,5 +13,6 @@
         </hardware>
       </xacro:if>
-      <xacro:unless value="$(arg use_sim)">
+      <xacro:unless
+        value="$(arg use_sim)">
         <hardware>
           <xacro:if value="${use_fake_hardware}">
@@ -25,17 +26,32 @@
         </hardware>
       </xacro:unless>
-      <joint name="axis_e">
-        <command_interface name="position" />
-        <command_interface name="velocity" />
+      <joint
+        name="axis_a">
+        <command_interface name="position">
+          <param name="min">0</param>
+          <param name="max">0.015</param>
+        </command_interface>
+        <command_interface name="velocity">
+          <param name="min">-2.5</param>
+          <param name="max">2.5</param>
+        </command_interface>
         <state_interface name="position">
           <param name="initial_value">${initial_positions['axis_e']}</param>
         </state_interface>
-        <state_interface name="velocity">
+        <state_interface
+          name="velocity">
           <param name="initial_value">${initial_velocities['axis_e']}</param>
         </state_interface>
       </joint>
-      <joint name="axis_d">
-        <command_interface name="position" />
-        <command_interface name="velocity" />
+      <joint
+        name="axis_b">
+        <command_interface name="position">
+          <param name="min">0</param>
+          <param name="max">3.22</param>
+        </command_interface>
+        <command_interface name="velocity">
+          <param name="min">-1.0</param>
+          <param name="max">1.0</param>
+        </command_interface>
         <state_interface name="position">
           <param name="initial_value">${initial_positions['axis_d']}</param>
@@ -45,7 +61,14 @@
         </state_interface>
       </joint>
-      <joint name="axis_c">
-        <command_interface name="position" />
-        <command_interface name="velocity" />
+      <joint
+        name="axis_c">
+        <command_interface name="position">
+          <param name="min">0</param>
+          <param name="max">3.22</param>
+        </command_interface>
+        <command_interface name="velocity">
+          <param name="min">-1.0</param>
+          <param name="max">1.0</param>
+        </command_interface>
         <state_interface name="position">
           <param name="initial_value">${initial_positions['axis_c']}</param>
@@ -55,7 +78,14 @@
         </state_interface>
       </joint>
-      <joint name="axis_b">
-        <command_interface name="position" />
-        <command_interface name="velocity" />
+      <joint
+        name="axis_d">
+        <command_interface name="position">
+          <param name="min">0</param>
+          <param name="max">3.49</param>
+        </command_interface>
+        <command_interface name="velocity">
+          <param name="min">-1.0</param>
+          <param name="max">1.0</param>
+        </command_interface>
         <state_interface name="position">
           <param name="initial_value">${initial_positions['axis_b']}</param>
@@ -65,7 +95,14 @@
         </state_interface>
       </joint>
-      <joint name="axis_a">
-        <command_interface name="position" />
-        <command_interface name="velocity" />
+      <joint
+        name="axis_e">
+        <command_interface name="position">
+          <param name="min">0</param>
+          <param name="max">6.10</param>
+        </command_interface>
+        <command_interface name="velocity">
+          <param name="min">-0.5</param>
+          <param name="max">0.5</param>
+        </command_interface>
         <state_interface name="position">
           <param name="initial_value">${initial_positions['axis_a']}</param>

File: alpha_description/srdf/alpha.srdf.xacro (robot description, xacro)
@@ -4,15 +4,15 @@
         <group name="${prefix}alpha">
             <link name="${prefix}ee_base_link" />
+            <joint name="${prefix}axis_a" />
+            <joint name="${prefix}axis_b" />
+            <joint name="${prefix}axis_c" />
+            <joint name="${prefix}axis_d" />
             <joint name="${prefix}axis_e" />
-            <joint name="${prefix}axis_d" />
-            <joint name="${prefix}axis_c" />
-            <joint name="${prefix}axis_b" />
-            <joint name="${prefix}axis_a" />
         </group>
         <group_state name="home" group="${prefix}alpha">
             <joint name="${prefix}axis_a" value="0" />
-            <joint name="${prefix}axis_b" value="1.5746" />
-            <joint name="${prefix}axis_c" value="0" />
-            <joint name="${prefix}axis_d" value="0" />
+            <joint name="${prefix}axis_b" value="0" />
+            <joint name="${prefix}axis_c" value="0.08" />
+            <joint name="${prefix}axis_d" value="1.5746" />
             <joint name="${prefix}axis_e" value="0" />
         </group_state>

File: alpha_description/urdf/alpha.urdf.xacro (robot description, xacro)
@@ -63,5 +63,5 @@
       </inertial>
     </link>
-    <joint name="${prefix}axis_a" type="revolute">
+    <joint name="${prefix}axis_e" type="revolute">
       <parent link="${prefix}m3_inline_link" />
       <child link="${prefix}m2_1_1_link" />
@@ -105,5 +105,5 @@
       </inertial>
     </link>
-    <joint name="${prefix}axis_b" type="revolute">
+    <joint name="${prefix}axis_d" type="revolute">
       <parent link="${prefix}m2_1_1_link" />
       <child link="${prefix}m2_joint_link" />
@@ -166,5 +166,5 @@
       </inertial>
     </link>
-    <joint name="${prefix}axis_d" type="revolute">
+    <joint name="${prefix}axis_b" type="revolute">
       <parent link="${prefix}m2_1_2_link" />
       <child link="${prefix}m1_link" />
@@ -195,5 +195,5 @@
       </inertial>
     </link>
-    <joint name="${prefix}axis_e" type="prismatic">
+    <joint name="${prefix}axis_a" type="prismatic">
       <origin rpy="0 0 0" xyz="0 0 0.009" />
       <parent link="${prefix}ee_base_link" />
@@ -206,5 +206,5 @@
     <xacro:alpha_standard_jaws parent="${prefix}ee_base_link"
       prefix="${prefix}standard_jaws_"
-      axis_a="${prefix}axis_e">
+      axis_a="${prefix}axis_a">
       <origin xyz="0 0 0" rpy="0 0 0" />
     </xacro:alpha_standard_jaws>
