Commit message: Added base platform option

File: alpha_description/xacro/alpha.urdf.xacro (robot description, xacro)
@@ -214,5 +214,4 @@
       <parent link="${parent}" />
       <child link="${prefix}base_link" />
-      <xacro:insert_block name="origin" />
     </joint>
     <joint name="${prefix}base_link_joint" type="fixed">

File: alpha_description/xacro/alpha_platform.config.xacro (robot description, xacro)
@@ -16,11 +16,12 @@
   <xacro:property name="use_sim" value="$(arg use_sim)" />
   <!-- Imports -->
-  <xacro:include filename="$(find ${description_package})/xacro/alpha.urdf.xacro" />
+  <xacro:include filename="$(find ${description_package})/xacro/alpha_platform.urdf.xacro" />
   <xacro:include filename="$(find ${description_package})/xacro/alpha.ros2_control.xacro" />
-  <link name="base_footprint" />
-  <xacro:alpha_urdf parent="base_footprint" prefix="${prefix}"
+  <!-- Define a world frame for Moveit -->
+  <link name="world" />
+  <xacro:alpha_platform_urdf prefix="${prefix}" parent="world"
     description_package="${description_package}">
-    <origin xyz="0 0 0" rpy="0 0 0" />
-  </xacro:alpha_urdf>
+    <origin xyz="0 0 0.06" rpy="0 0 0" />
+  </xacro:alpha_platform_urdf>
   <xacro:alpha_system prefix="${prefix}" name="ReachAlpha5" serial_port="$(arg serial_port)"
     state_update_frequency="$(arg state_update_frequency)"
