Commit message: Fixed naming errors

File: alpha_description/xacro/alpha.config.xacro (robot description, xacro)
@@ -32,5 +32,5 @@
   <xacro:if value="${use_sim}">
     <xacro:include filename="$(find ${description_package})/xacro/alpha.gazebo.xacro" />
-    <xacro:angler_gazebo prefix="${prefix}" description_package="${description_package}"
+    <xacro:alpha_gazebo prefix="${prefix}" description_package="${description_package}"
       namespace="$(arg namespace)"
       controllers_file="$(arg controllers_file)" />

File: alpha_description/xacro/alpha.gazebo.xacro (robot description, xacro)
@@ -1,5 +1,5 @@
 <?xml version="1.0"?>
 <robot xmlns:xacro="http://www.ros.org/wiki/xacro">
-  <xacro:macro name="angler_gazebo"
+  <xacro:macro name="alpha_gazebo"
     params="
       prefix

File: alpha_description/xacro/alpha_platform.config.xacro (robot description, xacro)
@@ -33,5 +33,5 @@
   <xacro:if value="${use_sim}">
     <xacro:include filename="$(find ${description_package})/xacro/alpha.gazebo.xacro" />
-    <xacro:angler_gazebo prefix="${prefix}" description_package="${description_package}"
+    <xacro:alpha_gazebo prefix="${prefix}" description_package="${description_package}"
       namespace="$(arg namespace)"
       controllers_file="$(arg controllers_file)" />

Commit message: wip: Started integrating mimic joints

File: alpha_description/xacro/alpha.config.xacro (robot description, xacro)
@@ -15,16 +15,25 @@
   <xacro:property name="prefix" value="$(arg prefix)" />
   <xacro:property name="use_sim" value="$(arg use_sim)" />
+  <xacro:property name="ee_prefix" value="standard_jaws_" />
   <!-- Imports -->
   <xacro:include filename="$(find ${description_package})/xacro/alpha.urdf.xacro" />
   <xacro:include filename="$(find ${description_package})/xacro/alpha.ros2_control.xacro" />
   <link name="base_footprint" />
-  <xacro:alpha_urdf parent="base_footprint" prefix="${prefix}"
+  <xacro:alpha_urdf
+    parent="base_footprint"
+    prefix="${prefix}"
+    ee_prefix="${ee_prefix}"
     description_package="${description_package}">
     <origin xyz="0 0 0" rpy="0 0 0" />
   </xacro:alpha_urdf>
-  <xacro:alpha_system prefix="${prefix}" name="ReachAlpha5" serial_port="$(arg serial_port)"
+  <xacro:alpha_system
+    prefix="${prefix}"
+    ee_prefix="${ee_prefix}"
+    name="ReachAlpha5"
+    serial_port="$(arg serial_port)"
     state_update_frequency="$(arg state_update_frequency)"
     initial_positions_file="$(arg initial_positions_file)"
-    description_package="${description_package}" use_sim="${use_sim}"
+    description_package="${description_package}"
+    use_sim="${use_sim}"
     use_fake_hardware="$(arg use_fake_hardware)"
   />
@@ -32,5 +41,7 @@
   <xacro:if value="${use_sim}">
     <xacro:include filename="$(find ${description_package})/xacro/alpha.gazebo.xacro" />
-    <xacro:alpha_gazebo prefix="${prefix}" description_package="${description_package}"
+    <xacro:alpha_gazebo
+      prefix="${prefix}"
+      description_package="${description_package}"
       namespace="$(arg namespace)"
       controllers_file="$(arg controllers_file)" />

File: alpha_description/xacro/alpha.gazebo.xacro (robot description, xacro)
@@ -4,4 +4,5 @@
     params="
       prefix
+      ee_prefix
       description_package
       namespace
@@ -21,36 +22,36 @@
     </gazebo>
     <!-- Materials -->
-    <gazebo reference="${prefix}alpha_base_link">
+    <gazebo reference="${prefix}base_link">
       <material>Gazebo/Gray</material>
     </gazebo>
-    <gazebo reference="${prefix}alpha_ee_base_link">
+    <gazebo reference="${prefix}ee_base_link">
       <material>Gazebo/Gray</material>
     </gazebo>
-    <gazebo reference="${prefix}alpha_m1_link" />
-    <gazebo reference="${prefix}alpha_m1_link">
+    <gazebo reference="${prefix}m1_link" />
+    <gazebo reference="${prefix}m1_link">
       <material>Gazebo/Gray</material>
     </gazebo>
-    <gazebo reference="${prefix}alpha_m2_1_1_link">
+    <gazebo reference="${prefix}m2_1_1_link">
       <material>Gazebo/Gray</material>
     </gazebo>
-    <gazebo reference="${prefix}alpha_m2_1_2_link">
+    <gazebo reference="${prefix}m2_1_2_link">
       <material>Gazebo/Gray</material>
     </gazebo>
-    <gazebo reference="${prefix}alpha_m2_joint_link">
+    <gazebo reference="${prefix}m2_joint_link">
       <material>Gazebo/Gray</material>
     </gazebo>
-    <gazebo reference="${prefix}alpha_m3_inline_link">
+    <gazebo reference="${prefix}m3_inline_link">
       <material>Gazebo/Gray</material>
     </gazebo>
-    <gazebo reference="${prefix}alpha_push_rod">
+    <gazebo reference="${prefix}push_rod">
       <material>Gazebo/Gray</material>
     </gazebo>
-    <gazebo reference="${prefix}alpha_standard_jaws_base_link">
+    <gazebo reference="${prefix}${ee_prefix}base_link">
       <material>Gazebo/Gray</material>
     </gazebo>
-    <gazebo reference="${prefix}alpha_standard_jaws_rs1_130_link">
+    <gazebo reference="${prefix}${ee_prefix}rs1_130_link">
       <material>Gazebo/Gray</material>
     </gazebo>
-    <gazebo reference="${prefix}alpha_standard_jaws_rs1_139_link">
+    <gazebo reference="${prefix}${ee_prefix}rs1_139_link">
       <material>Gazebo/Gray</material>
     </gazebo>

File: alpha_description/xacro/alpha.ros2_control.xacro (robot description, xacro)
@@ -4,4 +4,5 @@
     params="
       prefix
+      ee_prefix
       name
       serial_port
@@ -18,4 +19,23 @@
           <plugin>gz_ros2_control/GazeboSimSystem</plugin>
         </hardware>
+        <!-- Setup the mimic joints for simulation -->
+        <joint name="${prefix}${ee_prefix}rs1_130_joint">
+          <param name="mimic">${prefix}axis_a</param>
+          <param name="multiplier">51</param>
+          <param name="offset">0</param>
+          <command_interface name="position" />
+          <command_interface name="velocity" />
+          <state_interface name="position" />
+          <state_interface name="velocity" />
+        </joint>
+        <joint name="${prefix}${ee_prefix}rs1_139_joint">
+          <param name="mimic">${prefix}${ee_prefix}rs1_130_joint</param>
+          <param name="multiplier">1</param>
+          <param name="offset">0</param>
+          <command_interface name="position" />
+          <command_interface name="velocity" />
+          <state_interface name="position" />
+          <state_interface name="velocity" />
+        </joint>
       </xacro:if>
       <xacro:unless

File: alpha_description/xacro/alpha.urdf.xacro (robot description, xacro)
@@ -1,5 +1,11 @@
 <?xml version="1.0"?>
 <robot xmlns:xacro="http://ros.org/wiki/xacro">
-  <xacro:macro name="alpha_urdf" params="parent prefix description_package *origin">
+  <xacro:macro name="alpha_urdf"
+    params="
+      parent
+      prefix
+      ee_prefix
+      description_package
+      *origin">
     <material name="${prefix}black">
       <color rgba="0.3 0.3 0.3 1" />
@@ -173,10 +179,4 @@
     </link>
     <link name="${prefix}ee_base_link">
-      <visual>
-        <origin rpy="0 0 0" xyz="0 0 0" />
-        <geometry>
-          <box size="0.001 0.001 0.001" />
-        </geometry>
-      </visual>
       <inertial>
         <mass value="0.0001" />
@@ -192,10 +192,4 @@
     </link>
     <link name="${prefix}push_rod">
-      <visual>
-        <origin rpy="0 0 0" xyz="0 0 0" />
-        <geometry>
-          <box size="0.001 0.001 0.001" />
-        </geometry>
-      </visual>
       <inertial>
         <mass value="0.0001" />
@@ -264,5 +258,5 @@
       filename="$(find ${description_package})/xacro/end_effectors/standard_jaws.urdf.xacro" />
     <xacro:standard_jaws parent="${prefix}ee_base_link"
-      prefix="${prefix}standard_jaws_"
+      prefix="${prefix}${ee_prefix}"
       axis_a="${prefix}axis_a" description_package="${description_package}">
       <origin xyz="0 0 0" rpy="0 0 0" />

File: alpha_description/xacro/alpha_platform.config.xacro (robot description, xacro)
@@ -15,4 +15,5 @@
   <xacro:property name="prefix" value="$(arg prefix)" />
   <xacro:property name="use_sim" value="$(arg use_sim)" />
+  <xacro:property name="ee_prefix" value="standard_jaws_" />
   <!-- Imports -->
   <xacro:include filename="$(find ${description_package})/xacro/alpha_platform.urdf.xacro" />
@@ -20,9 +21,16 @@
   <!-- Define a world frame for Moveit -->
   <link name="world" />
-  <xacro:alpha_platform_urdf prefix="${prefix}" parent="world"
+  <xacro:alpha_platform_urdf
+    prefix="${prefix}"
+    ee_prefix="${ee_prefix}"
+    parent="world"
     description_package="${description_package}">
     <origin xyz="0 0 0.06" rpy="0 0 0" />
   </xacro:alpha_platform_urdf>
-  <xacro:alpha_system prefix="${prefix}" name="ReachAlpha5" serial_port="$(arg serial_port)"
+  <xacro:alpha_system
+    prefix="${prefix}"
+    ee_prefix="${ee_prefix}"
+    name="ReachAlpha5"
+    serial_port="$(arg serial_port)"
     state_update_frequency="$(arg state_update_frequency)"
     initial_positions_file="$(arg initial_positions_file)"
@@ -33,5 +41,8 @@
   <xacro:if value="${use_sim}">
     <xacro:include filename="$(find ${description_package})/xacro/alpha.gazebo.xacro" />
-    <xacro:alpha_gazebo prefix="${prefix}" description_package="${description_package}"
+    <xacro:alpha_gazebo
+      prefix="${prefix}"
+      ee_prefix="${ee_prefix}"
+      description_package="${description_package}"
       namespace="$(arg namespace)"
       controllers_file="$(arg controllers_file)" />

File: alpha_description/xacro/alpha_platform.urdf.xacro (robot description, xacro)
@@ -1,5 +1,11 @@
 <?xml version="1.0"?>
 <robot name="alpha_platform_urdf" xmlns:xacro="http://ros.org/wiki/xacro">
-  <xacro:macro name="alpha_platform_urdf" params="parent prefix description_package *origin">
+  <xacro:macro name="alpha_platform_urdf"
+    params="
+      parent
+      prefix
+      ee_prefix
+      description_package
+      *origin">
     <!-- Define a base platform for the alpha -->
     <link name="${prefix}platform">
@@ -29,5 +35,8 @@
     </joint>
     <xacro:include filename="$(find ${description_package})/xacro/alpha.urdf.xacro" />
-    <xacro:alpha_urdf parent="${prefix}base_footprint" prefix="${prefix}"
+    <xacro:alpha_urdf
+      parent="${prefix}base_footprint"
+      prefix="${prefix}"
+      ee_prefix="${ee_prefix}"
       description_package="${description_package}">
       <origin xyz="0 0 0" rpy="0 0 0" />
