Commit message: Added urdf specifications and rviz launch

File: alpha_description/urdf/alpha.urdf.xacro (robot description, xacro)
@@ -2,5 +2,5 @@
 <robot name="alpha_5_example" xmlns:xacro="http://ros.org/wiki/xacro">
   <xacro:include
-    filename="$(find bpl_alpha_description)/urdf/alpha_5_description.urdf.xacro" />
+    filename="$(find alpha_description)/urdf/alpha_description.urdf.xacro" />
   <link name="base_link" />
   <xacro:alpha_5 parent="base_link" name="alpha">

File: alpha_description/urdf/alpha_description.urdf.xacro (robot description, xacro)
@@ -15,5 +15,5 @@
       <visual>
         <geometry>
-          <mesh filename="package://bpl_alpha_description/meshes/M3-INLINE.stl" />
+          <mesh filename="package://alpha_description/meshes/M3-INLINE.stl" />
         </geometry>
         <origin rpy="0 0 0" xyz="0 0 0" />
@@ -35,5 +35,5 @@
       <visual>
         <geometry>
-          <mesh filename="package://bpl_alpha_description/meshes/M2-1-1.stl" />
+          <mesh filename="package://alpha_description/meshes/M2-1-1.stl" />
         </geometry>
         <origin rpy="0 0 0" xyz="0 0 0" />
@@ -57,5 +57,5 @@
       <visual>
         <geometry>
-          <mesh filename="package://bpl_alpha_description/meshes/M2.stl" />
+          <mesh filename="package://alpha_description/meshes/M2.stl" />
         </geometry>
         <origin rpy="0 0 0" xyz="0 0 0" />
@@ -91,5 +91,5 @@
       <visual>
         <geometry>
-          <mesh filename="package://bpl_alpha_description/meshes/M2-1-3.stl" />
+          <mesh filename="package://alpha_description/meshes/M2-1-3.stl" />
         </geometry>
         <origin rpy="0 0 0" xyz="0 0 0" />
@@ -114,5 +114,5 @@
         <geometry>
           <mesh
-            filename="package://bpl_alpha_description/meshes/RS1-100-101-123.stl" />
+            filename="package://alpha_description/meshes/RS1-100-101-123.stl" />
         </geometry>
         <origin rpy="0 -1.5707 0" xyz="0 0 0" />
@@ -152,5 +152,5 @@
     </joint>
     <xacro:include
-      filename="$(find bpl_alpha_description)/urdf/end_effectors/standard_jaws.urdf.xacro" />
+      filename="$(find alpha_description)/urdf/end_effectors/standard_jaws.urdf.xacro" />
     <xacro:alpha_standard_jaws parent="${name}_jaws_base_link"
       name="${name}_standard_jaws" axis_a="${name}_axis_a">

File: alpha_description/urdf/end_effectors/standard_jaws.urdf.xacro (robot description, xacro)
@@ -16,5 +16,5 @@
         <geometry>
           <mesh
-            filename="package://bpl_alpha_description/meshes/end_effectors/RS1-124.stl" />
+            filename="package://alpha_description/meshes/end_effectors/RS1-124.stl" />
         </geometry>
         <material name="${name}_black" />
@@ -25,5 +25,5 @@
         <geometry>
           <mesh
-            filename="package://bpl_alpha_description/meshes/end_effectors/RS1-130.stl" />
+            filename="package://alpha_description/meshes/end_effectors/RS1-130.stl" />
         </geometry>
         <material name="${name}_black" />
@@ -49,5 +49,5 @@
         <geometry>
           <mesh
-            filename="package://bpl_alpha_description/meshes/end_effectors/RS1-139.stl" />
+            filename="package://alpha_description/meshes/end_effectors/RS1-139.stl" />
         </geometry>
         <material name="${name}_black" />

Commit message: starting integration of ros2_control xacro

File: alpha_description/urdf/alpha.urdf.xacro (robot description, xacro)
@@ -4,6 +4,6 @@
     filename="$(find alpha_description)/urdf/alpha_description.urdf.xacro" />
   <link name="base_link" />
-  <xacro:alpha_5 parent="base_link" name="alpha">
+  <xacro:alpha parent="base_link" name="alpha">
     <origin xyz="0 0 0" rpy="0 0 0" />
-  </xacro:alpha_5>
+  </xacro:alpha>
 </robot>

File: alpha_description/urdf/alpha_description.urdf.xacro (robot description, xacro)
@@ -1,5 +1,5 @@
 <?xml version="1.0"?>
-<robot name="alpha_5" xmlns:xacro="http://ros.org/wiki/xacro">
-  <xacro:macro name="alpha_5" params="parent *origin name:=alpha_5">
+<robot name="alpha" xmlns:xacro="http://ros.org/wiki/xacro">
+  <xacro:macro name="alpha" params="parent *origin name:=alpha">
     <joint name="${name}_joint" type="fixed">
       <xacro:insert_block name="origin" />

Commit message: added ros2_control descriptions nad config and gazebo macro

File: alpha_description/urdf/alpha.urdf.xacro (robot description, xacro)
@@ -1,9 +1,37 @@
 <?xml version="1.0"?>
-<robot name="alpha_5_example" xmlns:xacro="http://ros.org/wiki/xacro">
+<robot name="alpha" xmlns:xacro="http://ros.org/wiki/xacro">
+  <!-- Declare arguments which can be set from a launch file -->
+  <xacro:arg name="prefix" default="" />
+  <xacro:arg name="use_gazebo" default="true" />
+  <xacro:arg name="use_fake_hardware" default="true" />
+  <xacro:arg name="mock_sensor_commands" default="true" />
+  <xacro:arg name="serial_port" default="" />
+  <xacro:arg name="heartbeat_timeout" default="5000" />
+  <xacro:arg name="state_update_frequency" default="200" />
+  <!-- Import Alpha macro -->
   <xacro:include
     filename="$(find alpha_description)/urdf/alpha_description.urdf.xacro" />
-  <link name="base_link" />
-  <xacro:alpha parent="base_link" name="alpha">
+  <!-- Import ros2_control macro -->
+  <xacro:include
+    filename="$(find alpha_description)/ros2_control/alpha.ros2_control.xacro" />
+  <xacro:if value="$(arg use_gazebo)">
+    <xacro:include
+      filename="$(find alpha_description)/gazebo/alpha.gazebo.xacro" />
+  </xacro:if>
+  <link name="world" />
+  <xacro:alpha_robot parent="world" prefix="$(arg prefix)">
     <origin xyz="0 0 0" rpy="0 0 0" />
-  </xacro:alpha>
+  </xacro:alpha_robot>
+  <xacro:alpha_system prefix="$(arg prefix)"
+    use_fake_hardware="$(arg use_fake_hardware)"
+    mock_sensor_commands="$(arg mock_sensor_commands)"
+    serial_port="$(arg serial_port)"
+    heartbeat_timeout="$(arg heartbeat_timeout)"
+    state_update_frequency="$(arg state_update_frequency)" />
+  <xacro:if value="$(arg use_gazebo)">
+    <gazebo reference="world">
+      <static>true</static>
+    </gazebo>
+    <xacro:alpha_gazebo prefix="$(arg prefix)" />
+  </xacro:if>
 </robot>

File: alpha_description/urdf/alpha_description.urdf.xacro (robot description, xacro)
@@ -1,16 +1,16 @@
 <?xml version="1.0"?>
-<robot name="alpha" xmlns:xacro="http://ros.org/wiki/xacro">
-  <xacro:macro name="alpha" params="parent *origin name:=alpha">
-    <joint name="${name}_joint" type="fixed">
+<robot xmlns:xacro="http://ros.org/wiki/xacro">
+  <xacro:macro name="alpha_robot" params="parent prefix *origin">
+    <joint name="${prefix}base_joint" type="fixed">
       <xacro:insert_block name="origin" />
       <parent link="${parent}" />
-      <child link="${name}_base_link" />
+      <child link="${prefix}base_link" />
       <origin xyz="0 0 0" rpy="0 0 0" />
     </joint>
-    <material name="alpha_black">
+    <material name="${prefix}black">
       <color rgba="0.3 0.3 0.3 1" />
     </material>
-    <link name="${name}_base_link" />
-    <link name="${name}_m3_inline_link">
+    <link name="${prefix}base_link" />
+    <link name="${prefix}m3_inline_link">
       <visual>
         <geometry>
@@ -18,5 +18,5 @@
         </geometry>
         <origin rpy="0 0 0" xyz="0 0 0" />
-        <material name="alpha_black" />
+        <material name="${prefix}black" />
       </visual>
       <collision>
@@ -27,10 +27,10 @@
       </collision>
     </link>
-    <joint name="${name}_base_link_joint" type="fixed">
-      <parent link="${name}_base_link" />
-      <child link="${name}_m3_inline_link" />
+    <joint name="${prefix}base_link_joint" type="fixed">
+      <parent link="${prefix}base_link" />
+      <child link="${prefix}m3_inline_link" />
       <origin rpy="0 0 0" />
     </joint>
-    <link name="${name}_m2_1_1_link">
+    <link name="${prefix}m2_1_1_link">
       <visual>
         <geometry>
@@ -38,5 +38,5 @@
         </geometry>
         <origin rpy="0 0 0" xyz="0 0 0" />
-        <material name="${name}_black" />
+        <material name="${prefix}black" />
       </visual>
       <collision>
@@ -47,12 +47,12 @@
       </collision>
     </link>
-    <joint name="${name}_axis_e" type="revolute">
-      <parent link="${name}_m3_inline_link" />
-      <child link="${name}_m2_1_1_link" />
+    <joint name="${prefix}axis_e" type="revolute">
+      <parent link="${prefix}m3_inline_link" />
+      <child link="${prefix}m2_1_1_link" />
       <origin xyz="0 0 0.014" />
       <axis xyz="0 0 1" />
       <limit effort="9.0" lower="0.0" upper="6.3" velocity="0.5" />
     </joint>
-    <link name="${name}_m2_joint_link">
+    <link name="${prefix}m2_joint_link">
       <visual>
         <geometry>
@@ -60,5 +60,5 @@
         </geometry>
         <origin rpy="0 0 0" xyz="0 0 0" />
-        <material name="${name}_black" />
+        <material name="${prefix}black" />
       </visual>
       <collision>
@@ -81,12 +81,12 @@
       </collision>
     </link>
-    <joint name="${name}_axis_d" type="revolute">
-      <parent link="${name}_m2_1_1_link" />
-      <child link="${name}_m2_joint_link" />
+    <joint name="${prefix}axis_d" type="revolute">
+      <parent link="${prefix}m2_1_1_link" />
+      <child link="${prefix}m2_joint_link" />
       <origin xyz="-0.02 0 0.033" />
       <axis xyz="0 1 0" />
       <limit effort="9.0" lower="0.0" upper="3.8" velocity="0.5" />
     </joint>
-    <link name="${name}_m2_1_2_link">
+    <link name="${prefix}m2_1_2_link">
       <visual>
         <geometry>
@@ -94,5 +94,5 @@
         </geometry>
         <origin rpy="0 0 0" xyz="0 0 0" />
-        <material name="${name}_black" />
+        <material name="${prefix}black" />
       </visual>
       <collision>
@@ -103,12 +103,12 @@
       </collision>
     </link>
-    <joint name="${name}_axis_c" type="revolute">
-      <parent link="${name}_m2_joint_link" />
-      <child link="${name}_m2_1_2_link" />
+    <joint name="${prefix}axis_c" type="revolute">
+      <parent link="${prefix}m2_joint_link" />
+      <child link="${prefix}m2_1_2_link" />
       <origin xyz="-0.04 0 -0.1453" rpy="0 0 3.14159" />
       <axis xyz="0 1 0" />
       <limit effort="9.0" lower="0.0" upper="3.5" velocity="0.5" />
     </joint>
-    <link name="${name}_m1_link">
+    <link name="${prefix}m1_link">
       <visual>
         <geometry>
@@ -117,5 +117,5 @@
         </geometry>
         <origin rpy="0 -1.5707 0" xyz="0 0 0" />
-        <material name="${name}_black" />
+        <material name="${prefix}black" />
       </visual>
       <collision>
@@ -126,26 +126,25 @@
       </collision>
     </link>
-    <joint name="${name}_axis_b" type="revolute">
-      <parent link="${name}_m2_1_2_link" />
-      <child link="${name}_m1_link" />
+    <joint name="${prefix}axis_b" type="revolute">
+      <parent link="${prefix}m2_1_2_link" />
+      <child link="${prefix}m1_link" />
       <origin xyz="0.02 0 0.033" rpy="0 0 2.09439" />
       <axis xyz="0 0 -1" />
       <limit effort="9.0" lower="0.0" upper="6.2" velocity="0.5" />
     </joint>
-    <material name="${name}_jaws_black">
+    <material name="${prefix}jaws_black">
       <color rgba="0.3 0.3 0.3 1" />
     </material>
-    <joint name="${name}_jaws_joint" type="fixed">
+    <joint name="${prefix}jaws_joint" type="fixed">
       <origin rpy="0 0 0" xyz="0 0 0.09975" />
-      <parent link="${name}_m1_link" />
-      <child link="${name}_jaws_base_link" />
+      <parent link="${prefix}m1_link" />
+      <child link="${prefix}jaws_base_link" />
     </joint>
-    <link name="${name}_jaws_base_link">
-    </link>
-    <link name="${name}_push_rod" />
-    <joint name="${name}_axis_a" type="prismatic">
+    <link name="${prefix}jaws_base_link" />
+    <link name="${prefix}push_rod" />
+    <joint name="${prefix}axis_a" type="prismatic">
       <origin rpy="0 0 0" xyz="0 0 0.009" />
-      <parent link="${name}_jaws_base_link" />
-      <child link="${name}_push_rod" />
+      <parent link="${prefix}jaws_base_link" />
+      <child link="${prefix}push_rod" />
       <axis xyz="0 0 1" />
       <limit effort="10" lower="0" upper="0.015" velocity="10" />
@@ -153,6 +152,7 @@
     <xacro:include
       filename="$(find alpha_description)/urdf/end_effectors/standard_jaws.urdf.xacro" />
-    <xacro:alpha_standard_jaws parent="${name}_jaws_base_link"
-      name="${name}_standard_jaws" axis_a="${name}_axis_a">
+    <xacro:alpha_standard_jaws parent="${prefix}jaws_base_link"
+      prefix="${prefix}jaws"
+      axis_a="${prefix}axis_a">
       <origin xyz="0 0 0" rpy="0 0 0" />
     </xacro:alpha_standard_jaws>

File: alpha_description/urdf/end_effectors/standard_jaws.urdf.xacro (robot description, xacro)
@@ -1,16 +1,16 @@
 <?xml version="1.0"?>
-<robot name="alpha_standard_jaws" xmlns:xacro="http://ros.org/wiki/xacro">
+<robot xmlns:xacro="http://ros.org/wiki/xacro">
   <xacro:macro name="alpha_standard_jaws"
-    params="parent *origin name:=alpha_standard_jaws axis_a">
-    <material name="${name}_black">
+    params="parent prefix axis_a *origin">
+    <material name="${prefix}black">
       <color rgba="0.3 0.3 0.3 1" />
     </material>
-    <joint name="${name}_joint" type="fixed">
+    <joint name="${prefix}base_joint" type="fixed">
       <xacro:insert_block name="origin" />
       <parent link="${parent}" />
-      <child link="${name}_base_link" />
+      <child link="${prefix}base_link" />
       <origin xyz="0 0 0" rpy="0 0 0" />
     </joint>
-    <link name="${name}_base_link">
+    <link name="${prefix}base_link">
       <visual>
         <geometry>
@@ -18,8 +18,8 @@
             filename="package://alpha_description/meshes/end_effectors/RS1-124.stl" />
         </geometry>
-        <material name="${name}_black" />
+        <material name="${prefix}black" />
       </visual>
     </link>
-    <link name="${name}_rs1_130_link">
+    <link name="${prefix}rs1_130_link">
       <visual>
         <geometry>
@@ -27,5 +27,5 @@
             filename="package://alpha_description/meshes/end_effectors/RS1-130.stl" />
         </geometry>
-        <material name="${name}_black" />
+        <material name="${prefix}black" />
         <origin xyz="0 0 0" rpy="0 0 0" />
       </visual>
@@ -37,13 +37,13 @@
       </collision>
     </link>
-    <joint name="${name}_rs1_130_joint" type="revolute">
+    <joint name="${prefix}rs1_130_joint" type="revolute">
       <origin xyz="0 0.0155 0.0069" rpy="0 0 0" />
-      <parent link="${name}_base_link" />
-      <child link="${name}_rs1_130_link" />
+      <parent link="${prefix}base_link" />
+      <child link="${prefix}rs1_130_link" />
       <axis xyz="-1 0 0" />
       <limit lower="0" upper="0.5" effort="10" velocity="10" />
       <mimic joint="${axis_a}" multiplier="51" offset="0" />
     </joint>
-    <link name="${name}_rs1_139_link">
+    <link name="${prefix}rs1_139_link">
       <visual>
         <geometry>
@@ -51,5 +51,5 @@
             filename="package://alpha_description/meshes/end_effectors/RS1-139.stl" />
         </geometry>
-        <material name="${name}_black" />
+        <material name="${prefix}black" />
         <origin xyz="0 0 0" rpy="0 0 0" />
       </visual>
@@ -61,11 +61,11 @@
       </collision>
     </link>
-    <joint name="${name}_rs1_139_joint" type="revolute">
+    <joint name="${prefix}rs1_139_joint" type="revolute">
       <origin xyz="0 -0.0155 0.0069" rpy="0 0 0" />
-      <parent link="${name}_base_link" />
-      <child link="${name}_rs1_139_link" />
+      <parent link="${prefix}base_link" />
+      <child link="${prefix}rs1_139_link" />
       <axis xyz="1 0 0" />
       <limit lower="0" upper="0.5" effort="10" velocity="10" />
-      <mimic joint="${name}_rs1_130_joint" multiplier="1" offset="0" />
+      <mimic joint="${prefix}rs1_130_joint" multiplier="1" offset="0" />
     </joint>
   </xacro:macro>

Commit message: Added documented inertial properties

File: alpha_description/urdf/alpha.urdf.xacro (robot description, xacro)
@@ -27,7 +27,10 @@
       </collision>
       <inertial>
-        <mass value="2e-06" />
-        <inertia ixx="1.1e-09" ixy="0" ixz="0" iyy="1.1e-09" iyz="0"
-          izz="1.1e-09" />
+        <mass value="0.341" />
+        <origin xyz="-0.075 -0.006 -0.003" />
+        <inertia
+          ixx="0.000099" ixy="0.000139" ixz="0.000115"
+          iyx="0.000139" iyy="0.00292" iyz="0.000003"
+          izx="0.000115" izy="0.000003" izz="0.002934" />
       </inertial>
     </link>
@@ -52,7 +55,10 @@
       </collision>
       <inertial>
-        <mass value="2e-06" />
-        <inertia ixx="1.1e-09" ixy="0" ixz="0" iyy="1.1e-09" iyz="0"
-          izz="1.1e-09" />
+        <mass value="0.194" />
+        <origin xyz="0.005 -0.001 0.016" />
+        <inertia
+          ixx="0.000189" ixy="0.000005" ixz="0.000054"
+          iyx="0.000005" iyy="0.000213" iyz="0.000003"
+          izx="0.000054" izy="0.000003" izz="0.000067" />
       </inertial>
     </link>
@@ -91,7 +97,10 @@
       </collision>
       <inertial>
-        <mass value="2e-06" />
-        <inertia ixx="1.1e-09" ixy="0" ixz="0" iyy="1.1e-09" iyz="0"
-          izz="1.1e-09" />
+        <mass value="0.429" />
+        <origin xyz="0.073 0.0 0.0" />
+        <inertia
+          ixx="0.000087" ixy="-0.000076" ixz="-0.00001"
+          iyx="-0.000076" iyy="0.00319" iyz="0"
+          izx="-0.00001" izy="0" izz="0.003212" />
       </inertial>
     </link>
@@ -118,7 +127,10 @@
       </collision>
       <inertial>
-        <mass value="2e-06" />
-        <inertia ixx="1.1e-09" ixy="0" ixz="0" iyy="1.1e-09" iyz="0"
-          izz="1.1e-09" />
+        <mass value="0.115" />
+        <origin xyz="0.017 -0.026 -0.002" />
+        <inertia
+          ixx="0.00012" ixy="-0.000061" ixz="-0.000001"
+          iyx="-0.000061" iyy="0.000062" iyz="0"
+          izx="-0.000001" izy="0" izz="0.000156" />
       </inertial>
     </link>
@@ -146,7 +158,10 @@
       </collision>
       <inertial>
-        <mass value="2e-06" />
-        <inertia ixx="1.1e-09" ixy="0" ixz="0" iyy="1.1e-09" iyz="0"
-          izz="1.1e-09" />
+        <mass value="0.333" />
+        <origin xyz="0.0 0.003 -0.098" />
+        <inertia
+          ixx="0.003709" ixy="0.000002" ixz="-0.000004"
+          iyx="0.000002" iyy="0.003734" iyz="0"
+          izx="-0.000004" izy="0" izz="0.000079" />
       </inertial>
     </link>

Commit message: resolved bugs in hardware configuration with moveit

File: alpha_description/urdf/alpha.urdf.xacro (robot description, xacro)
@@ -63,5 +63,5 @@
       </inertial>
     </link>
-    <joint name="${prefix}axis_e" type="revolute">
+    <joint name="${prefix}axis_a" type="revolute">
       <parent link="${prefix}m3_inline_link" />
       <child link="${prefix}m2_1_1_link" />
@@ -105,5 +105,5 @@
       </inertial>
     </link>
-    <joint name="${prefix}axis_d" type="revolute">
+    <joint name="${prefix}axis_b" type="revolute">
       <parent link="${prefix}m2_1_1_link" />
       <child link="${prefix}m2_joint_link" />
@@ -166,5 +166,5 @@
       </inertial>
     </link>
-    <joint name="${prefix}axis_b" type="revolute">
+    <joint name="${prefix}axis_d" type="revolute">
       <parent link="${prefix}m2_1_2_link" />
       <child link="${prefix}m1_link" />
@@ -195,5 +195,5 @@
       </inertial>
     </link>
-    <joint name="${prefix}axis_a" type="prismatic">
+    <joint name="${prefix}axis_e" type="prismatic">
       <origin rpy="0 0 0" xyz="0 0 0.009" />
       <parent link="${prefix}ee_base_link" />
@@ -206,5 +206,5 @@
     <xacro:alpha_standard_jaws parent="${prefix}ee_base_link"
       prefix="${prefix}standard_jaws_"
-      axis_a="${prefix}axis_a">
+      axis_a="${prefix}axis_e">
       <origin xyz="0 0 0" rpy="0 0 0" />
     </xacro:alpha_standard_jaws>

Commit message: Fix xacro compatibility for simulation

File: alpha_description/urdf/alpha.urdf.xacro (robot description, xacro)
@@ -15,5 +15,5 @@
       <visual>
         <geometry>
-          <mesh filename="package://alpha_description/meshes/M3-INLINE.stl" />
+          <mesh filename="file://$(find alpha_description)/meshes/M3-INLINE.stl" />
         </geometry>
         <origin rpy="0 0 0" xyz="0 0 0" />
@@ -43,5 +43,5 @@
       <visual>
         <geometry>
-          <mesh filename="package://alpha_description/meshes/M2-1-1.stl" />
+          <mesh filename="file://$(find alpha_description)/meshes/M2-1-1.stl" />
         </geometry>
         <origin rpy="0 0 0" xyz="0 0 0" />
@@ -73,5 +73,5 @@
       <visual>
         <geometry>
-          <mesh filename="package://alpha_description/meshes/M2.stl" />
+          <mesh filename="file://$(find alpha_description)/meshes/M2.stl" />
         </geometry>
         <origin rpy="0 0 0" xyz="0 0 0" />
@@ -115,5 +115,5 @@
       <visual>
         <geometry>
-          <mesh filename="package://alpha_description/meshes/M2-1-3.stl" />
+          <mesh filename="file://$(find alpha_description)/meshes/M2-1-3.stl" />
         </geometry>
         <origin rpy="0 0 0" xyz="0 0 0" />
@@ -146,5 +146,5 @@
         <geometry>
           <mesh
-            filename="package://alpha_description/meshes/RS1-100-101-123.stl" />
+            filename="file://$(find alpha_description)/meshes/RS1-100-101-123.stl" />
         </geometry>
         <origin rpy="0 -1.5707 0" xyz="0 0 0" />

File: alpha_description/urdf/end_effectors/standard_jaws.urdf.xacro (robot description, xacro)
@@ -16,5 +16,5 @@
         <geometry>
           <mesh
-            filename="package://alpha_description/meshes/end_effectors/RS1-124.stl" />
+            filename="file://$(find alpha_description)/meshes/end_effectors/RS1-124.stl" />
         </geometry>
         <material name="${prefix}black" />
@@ -30,5 +30,5 @@
         <geometry>
           <mesh
-            filename="package://alpha_description/meshes/end_effectors/RS1-130.stl" />
+            filename="file://$(find alpha_description)/meshes/end_effectors/RS1-130.stl" />
         </geometry>
         <material name="${prefix}black" />
@@ -59,5 +59,5 @@
         <geometry>
           <mesh
-            filename="package://alpha_description/meshes/end_effectors/RS1-139.stl" />
+            filename="file://$(find alpha_description)/meshes/end_effectors/RS1-139.stl" />
         </geometry>
         <material name="${prefix}black" />
